File: adpd1080_breakoutboard/power_in.kicad_sch (KiCad schematic)
At the start: 10 parts, among them J1 1V8_IN, J2 3V3_IN, J3 PG_TP, U1 LD39100 1V8

Commit message: replace txb0104 with txs0104e for i2c
- txb0104 does not work with i2c but txs0104e works
- changed the i2c pull-ups to 'no-placement' because
  the txs0104e has internal 10k pull-ups
- added test points for 1v8 logic scl and sda

Signed-off-by: Mika Laitio <lamikr@gmail.com>
Other:
- title: (none) -> ADPD1080 Breakoutboard
Changed lines of the file:
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@@
 	(generator_version "8.0")
 	(paper "A4")
+	(title_block
+		(title "ADPD1080 Breakoutboard")
+		(rev "v0.2")
+	)
 	(junction
 		(at 48.26 104.14)
